File: MechanicalDIY/MechanicalDIY.kicad_sch (KiCad schematic)
At the start: 163 parts, among them J1 OLED_128x64, SW1 RotaryEncoder_Switch, SW10 F9, SW11 F10, SW12 prtsc, SW13 F12, SW14 ., SW15 Tab, SW16 Caps, SW17 Shift, SW18 Ctrl, SW19 1, SW2 Esc, SW20 2, SW21 3, SW22 4, SW23 5, SW24 6, SW25 7, SW26 8, SW27 9, SW28 0, SW29 -, SW3 F1, SW30 =, SW31 Backspace, SW32 Q, SW33 W, SW34 E, SW35 R, SW36 T, SW37 Y, SW38 U, SW39 I, SW4 F2, SW40 O, SW41 P, SW42 [, SW43 ], SW44 \, SW45 A, SW46 S, SW47 D, SW48 F, SW49 G, SW5 F3, SW50 H, SW51 J, SW52 K, SW53 L, SW54 ;, SW55 ', SW56 Enter, SW57 Pause, SW58 Z, SW59 X, SW6 F5, SW60 C, SW61 V, SW62 B, SW63 N, SW64 M, SW65 <, SW66 >, SW67 ?, SW68 shift, SW69 Up, SW7 F6, SW70 delete, SW71 Win, SW72 Alt, SW73 Rigth, SW74 Down, SW75 left, SW76 Ctrl, SW77 Fn, SW78 Alt, SW79 Space, SW8 F7, SW9 Home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

Commit message: update
Parts:
- removed D27, D55, D66, D67, D68, D69, D70, D71, D72, D73, D74, D75, D76, D77, D78, D79, D80: ~, symbol ScottoKeebs:Placeholder_Diode
- removed F11: F11, symbol Switch:SW_Push_45deg
- removed F8: F8, symbol Switch:SW_Push_45deg
- removed SW1: RotaryEncoder_Switch, symbol Device:RotaryEncoder_Switch
- removed SW10: F9, symbol Switch:SW_Push_45deg
- removed SW11: F10, symbol Switch:SW_Push_45deg
- removed SW12: prtsc, symbol Switch:SW_Push_45deg
- removed SW13: F12, symbol Switch:SW_Push_45deg
- removed SW2: Esc, symbol Switch:SW_Push_45deg
- removed SW3: F1, symbol Switch:SW_Push_45deg
- removed SW4: F2, symbol Switch:SW_Push_45deg
- removed SW5: F3, symbol Switch:SW_Push_45deg
- removed SW6: F5, symbol Switch:SW_Push_45deg
- removed SW66: >, symbol Switch:SW_Push_45deg
- removed SW67: ?, symbol Switch:SW_Push_45deg
- removed SW68: shift, symbol Switch:SW_Push_45deg
- removed SW69: Up, symbol Switch:SW_Push_45deg
- removed SW7: F6, symbol Switch:SW_Push_45deg
- removed SW70: delete, symbol Switch:SW_Push_45deg
- removed SW71: Win, symbol Switch:SW_Push_45deg
- removed SW72, SW78: Alt, symbol Switch:SW_Push_45deg
- removed SW73: Rigth, symbol Switch:SW_Push_45deg
- removed SW74: Down, symbol Switch:SW_Push_45deg
- removed SW75: left, symbol Switch:SW_Push_45deg
- removed SW76: Ctrl, symbol Switch:SW_Push_45deg
- removed SW77: Fn, symbol Switch:SW_Push_45deg
- removed SW79: Space, symbol Switch:SW_Push_45deg
- removed SW8: F7, symbol Switch:SW_Push_45deg
- removed SW9: Home, symbol Switch:SW_Push_45deg
- removed U1: Raspberry_Pi_Pico, ScottoKeebs_MCU:Raspberry_Pi_Pico, symbol ScottoKeebs:MCU_Raspberry_Pi_Pico
- added BT1: Battery_Cell, symbol Device:Battery_Cell
- added D81, D82: ~, ScottoKeebs_Components:Diode_DO-35, symbol ScottoKeebs:Placeholder_Diode
- added H1, H2, H3, H4: MountingHole, MountingHole:MountingHole_3.2mm_M3, symbol Mechanical:MountingHole
- added J2: Conn_01x02_Pin, Connector_JST:JST_PH_S2B-PH-K_1x02_P2.00mm_Horizontal, symbol Connector:Conn_01x02_Pin
- added On1: SW_SPDT, Button_Switch_THT:SW_Slide_SPDT_Angled_CK_OS102011MA1Q, symbol Switch:SW_SPDT
- added SW19: R, ScottoKeebs_MX:MX_PCB_1.00u, symbol Switch:SW_Push_45deg
- added SW20: T, ScottoKeebs_MX:MX_PCB_1.00u, symbol Switch:SW_Push_45deg
- added SW21: Y, ScottoKeebs_MX:MX_PCB_1.00u, symbol Switch:SW_Push_45deg
- added SW22: U, ScottoKeebs_MX:MX_PCB_1.00u, symbol Switch:SW_Push_45deg
- added SW23: I, ScottoKeebs_MX:MX_PCB_1.00u, symbol Switch:SW_Push_45deg
- added SW24: O, ScottoKeebs_MX:MX_PCB_1.00u, symbol Switch:SW_Push_45deg
- added SW25: P, ScottoKeebs_MX:MX_PCB_1.00u, symbol Switch:SW_Push_45deg
- added SW26: [, ScottoKeebs_MX:MX_PCB_1.00u, symbol Switch:SW_Push_45deg
- added SW27: ], ScottoKeebs_MX:MX_PCB_1.00u, symbol Switch:SW_Push_45deg
- added SW28: Backspace, ScottoKeebs_MX:MX_PCB_2.00u, symbol Switch:SW_Push_45deg
- added SW29: CASPLOCK, ScottoKeebs_MX:MX_PCB_1.75u, symbol Switch:SW_Push_45deg
- added SW30: A, ScottoKeebs_MX:MX_PCB_1.00u, symbol Switch:SW_Push_45deg
- added SW31: S, ScottoKeebs_MX:MX_PCB_1.00u, symbol Switch:SW_Push_45deg
- added U1: Nice_Nano_V2, ScottoKeebs_MCU:Nice_Nano_V2, symbol ScottoKeebs:MCU_Nice_Nano_V2
- D1, D10, D11, D12, D13, D14, D15, D16, D17, D18, D19, D2, D20, D21, D22, D23, D24, D25, D26, D28, D29, D3, D30, D31, D32, D33, D34, D35, D36, D37, D38, D39, D4, D40, D41, D42, D43, D44, D45, D46, D47, D48, D49, D5, D50, D51, D52, D53, D54, D56, D57, D58, D59, D6, D60, D61, D62, D63, D64, D65, D7, D8, D9: footprint (none) -> ScottoKeebs_Components:Diode_DO-35
- SW1: renamed from SW14; value . -> Esc; footprint (none) -> ScottoKeebs_MX:MX_PCB_1.00u
- SW10: renamed from SW27; value 9 -> 8; footprint (none) -> ScottoKeebs_MX:MX_PCB_1.00u
- SW11: renamed from SW28; value 0 -> 9; footprint (none) -> ScottoKeebs_MX:MX_PCB_1.00u
- SW12: renamed from SW29; value - -> 0; footprint (none) -> ScottoKeebs_MX:MX_PCB_1.00u
- SW13: renamed from SW30; value = -> -; footprint (none) -> ScottoKeebs_MX:MX_PCB_1.00u
- SW14: renamed from SW31; value Backspace -> =; footprint (none) -> ScottoKeebs_MX:MX_PCB_1.00u
- SW15: footprint (none) -> ScottoKeebs_MX:MX_PCB_1.50u
- SW16: value Caps -> Q; footprint (none) -> ScottoKeebs_MX:MX_PCB_1.00u
- SW17: value Shift -> W; footprint (none) -> ScottoKeebs_MX:MX_PCB_1.00u
- SW18: value Ctrl -> E; footprint (none) -> ScottoKeebs_MX:MX_PCB_1.00u
- SW2: renamed from SW19; value 1 -> .; footprint (none) -> ScottoKeebs_MX:MX_PCB_1.00u
- SW3: renamed from SW20; value 2 -> 1; footprint (none) -> ScottoKeebs_MX:MX_PCB_1.00u
- SW32: value Q -> D; footprint (none) -> ScottoKeebs_MX:MX_PCB_1.00u
- SW33: value W -> F; footprint (none) -> ScottoKeebs_MX:MX_PCB_1.00u
- SW34: value E -> G; footprint (none) -> ScottoKeebs_MX:MX_PCB_1.00u
- SW35: value R -> H; footprint (none) -> ScottoKeebs_MX:MX_PCB_1.00u
- SW36: value T -> J; footprint (none) -> ScottoKeebs_MX:MX_PCB_1.00u
- SW37: value Y -> K; footprint (none) -> ScottoKeebs_MX:MX_PCB_1.00u
- SW38: value U -> L; footprint (none) -> ScottoKeebs_MX:MX_PCB_1.00u
- SW39: value I -> ;; footprint (none) -> ScottoKeebs_MX:MX_PCB_1.00u
- SW4: renamed from SW21; value 3 -> 2; footprint (none) -> ScottoKeebs_MX:MX_PCB_1.00u
- SW40: value O -> '; footprint (none) -> ScottoKeebs_MX:MX_PCB_1.00u
- SW41: value P -> eNTER; footprint (none) -> ScottoKeebs_MX:MX_PCB_2.25u
- SW42: value [ -> \; footprint (none) -> ScottoKeebs_MX:MX_PCB_1.50u
- SW43: value ] -> SHIFT; footprint (none) -> ScottoKeebs_MX:MX_PCB_2.25u
- SW44: value \ -> Z; footprint (none) -> ScottoKeebs_MX:MX_PCB_1.00u
- SW45: value A -> X; footprint (none) -> ScottoKeebs_MX:MX_PCB_1.00u
- SW46: value S -> C; footprint (none) -> ScottoKeebs_MX:MX_PCB_1.00u
- SW47: value D -> V; footprint (none) -> ScottoKeebs_MX:MX_PCB_1.00u
- SW48: value F -> B; footprint (none) -> ScottoKeebs_MX:MX_PCB_1.00u
- SW49: value G -> N; footprint (none) -> ScottoKeebs_MX:MX_PCB_1.00u
- SW5: renamed from SW22; value 4 -> 3; footprint (none) -> ScottoKeebs_MX:MX_PCB_1.00u
- SW50: value H -> M; footprint (none) -> ScottoKeebs_MX:MX_PCB_1.00u
- SW51: value J -> ,; footprint (none) -> ScottoKeebs_MX:MX_PCB_1.00u
- SW52: value K -> .; footprint (none) -> ScottoKeebs_MX:MX_PCB_1.00u
- SW53: value L -> /; footprint (none) -> ScottoKeebs_MX:MX_PCB_1.00u
- SW54: value ; -> SHIFT; footprint (none) -> ScottoKeebs_MX:MX_PCB_1.75u
- SW55: value ' -> UP; footprint (none) -> ScottoKeebs_MX:MX_PCB_1.00u
- SW56: value Enter -> CTRL; footprint (none) -> ScottoKeebs_MX:MX_PCB_1.25u
- SW57: value Pause -> FN; footprint (none) -> ScottoKeebs_MX:MX_PCB_1.25u
- SW58: value Z -> WIN; footprint (none) -> ScottoKeebs_MX:MX_PCB_1.25u
- SW59: value X -> ALT; footprint (none) -> ScottoKeebs_MX:MX_PCB_6.25u
- SW6: renamed from SW23; value 5 -> 4; footprint (none) -> ScottoKeebs_MX:MX_PCB_1.00u
- SW60: value C -> SPACE; footprint (none) -> ScottoKeebs_MX:MX_PCB_1.00u
- SW61: value V -> ALT; footprint (none) -> ScottoKeebs_MX:MX_PCB_1.00u
- SW62: value B -> CTRL; footprint (none) -> ScottoKeebs_MX:MX_PCB_1.00u
- SW63: value N -> LEFT; footprint (none) -> ScottoKeebs_MX:MX_PCB_1.00u
- SW64: value M -> DOWN; footprint (none) -> ScottoKeebs_MX:MX_PCB_1.00u
- SW65: value < -> RIGTH; footprint (none) -> ScottoKeebs_MX:MX_PCB_1.00u
- SW7: renamed from SW24; value 6 -> 5; footprint (none) -> ScottoKeebs_MX:MX_PCB_1.00u
- SW8: renamed from SW25; value 7 -> 6; footprint (none) -> ScottoKeebs_MX:MX_PCB_1.00u
- SW9: renamed from SW26; value 8 -> 7; footprint (none) -> ScottoKeebs_MX:MX_PCB_1.00u
Connections:
- net at D2.2 (A): now also SW9.2
- net at SW17.2: now also D13.2 (A); no longer D57.2 (A)
- net Row3: now reaches D30.1 (K)
- net Row3: now also D28.1 (K), D29.1 (K), D31.1 (K), D32.1 (K), D33.1 (K), D34.1 (K), D35.1 (K), D36.1 (K), D37.1 (K), D38.1 (K), D39.1 (K), D40.1 (K), D41.1 (K), U1.7 (4)
- net at D30.2 (A): now also SW31.2; no longer SW43.2
- net Column9: now reaches SW60.1
- net Column9: now also SW37.1, SW51.1, SW9.1, SW23.1, U1.18 (19)
- net at D8.2 (A): now also SW3.2
- net Column11: now reaches SW39.1
- net Column11: now also SW11.1, SW53.1, SW62.1, SW25.1, U1.20 (21)
- net at D34.2 (A): now also SW35.2; no longer SW39.2
- net Column14: now reaches SW14.1
- net Column14: now also SW42.1, SW65.1, SW28.1, U1.27 (7)
- net Row4: now reaches D54.1 (K)
- net Row4: now also D42.1 (K), D43.1 (K), D44.1 (K), D45.1 (K), D46.1 (K), D47.1 (K), D48.1 (K), D49.1 (K), D50.1 (K), D51.1 (K), D52.1 (K), D53.1 (K), U1.8 (5)
- net at D54.2 (A): now also SW55.2; no longer SW46.2
- net Row5: now reaches D65.1 (K)
- net Row5: now also D56.1 (K), D57.1 (K), D58.1 (K), D59.1 (K), D60.1 (K), D61.1 (K), D62.1 (K), D63.1 (K), D64.1 (K), U1.9 (6)
- net at D40.2 (A): now also SW41.2; no longer SW33.2
- net Column6: now reaches SW6.1
- net Column6: now also SW34.1, SW48.1, SW20.1, U1.15 (14)
- net at SW6.2: now also D5.2 (A); no longer D18.2 (A)
- net Row2: now reaches D13.1 (K)
- net Row2: now also D11.1 (K), D12.1 (K), D14.1 (K), D15.1 (K), D16.1 (K), D17.1 (K), D18.1 (K), D19.1 (K), D20.1 (K), D21.1 (K), D22.1 (K), D81.1 (K), D82.1 (K), U1.2 (0)
- net at SW1.2: now also D10.2 (A); no longer D13.2 (A)
- net at SW53.2: now also D52.2 (A)
- net at SW56.2: now also D56.2 (A); no longer D44.2 (A)
- net at D11.2 (A): now also SW15.2
- net at D22.2 (A): now also SW26.2; no longer SW10.2
- net at D42.2 (A): now also SW43.2
- net at D19.2 (A): now also SW23.2; no longer SW7.2
- net Column2: now reaches SW44.1
- net Column2: now also SW16.1, SW2.1, SW57.1, SW30.1, U1.11 (8)
- net at SW44.2: now also D43.2 (A); no longer D29.2 (A)
- net Row1: now reaches D5.1 (K)
- net Row1: now also D1.1 (K), D10.1 (K), D2.1 (K), D23.1 (K), D24.1 (K), D25.1 (K), D26.1 (K), D3.1 (K), D4.1 (K), D6.1 (K), D7.1 (K), D8.1 (K), D9.1 (K), U1.1
- net at D28.2 (A): now also SW29.2
- net at SW18.2: now also D14.2 (A)
- net Column3: now reaches SW58.1
- net Column3: now also SW17.1, SW3.1, SW45.1, SW31.1, U1.12 (9)
- net at D53.2 (A): now also SW54.2; no longer SW47.2
- net at D31.2 (A): now also SW32.2; no longer SW42.2
- net at SW51.2: now also D50.2 (A); no longer D49.2 (A)
- net GND: now reaches J1.1 (GND)
- net GND: now also J2.1 (Pin_1), U1.3 (GND)
- net VCC: now reaches J1.2 (VCC)
- net VCC: now also On1.3 (C), U1.24 (B+)
- net SCL: now reaches J1.3 (SCL)
- net SCL: now also U1.6 (3)
- net SDA: now reaches J1.4 (SDA)
- net SDA: now also U1.5 (2)
- net at D46.2 (A): now also SW47.2; no longer SW54.2
- net at D45.2 (A): now also SW46.2; no longer SW55.2
- net at SW48.2: now also D47.2 (A); no longer D52.2 (A)
- net Column4: now reaches SW59.1
- net Column4: now also SW18.1, SW32.1, SW4.1, SW46.1, U1.13 (10)
- net at D9.2 (A): now also SW2.2
- net at SW34.2: now also D33.2 (A); no longer D39.2 (A)
- net at D3.2 (A): now also SW8.2
- net Column7: now reaches SW7.1
- net Column7: now also SW35.1, SW49.1, SW21.1, U1.16 (15)
- net at D38.2 (A): now also SW39.2; no longer SW35.2
- net at D1.2 (A): now also SW10.2
- net Column13: now reaches SW64.1
- net Column13: now also SW13.1, SW41.1, SW55.1, SW27.1, U1.26 (2)
- net at D32.2 (A): now also SW33.2; no longer SW41.2
- net at SW4.2: now also D7.2 (A); no longer D16.2 (A)
- net Column8: now reaches SW36.1
- net Column8: now also SW50.1, SW8.1, SW22.1, U1.17 (18)
- net at D37.2 (A): now also SW38.2; no longer SW36.2
- net Column10: now reaches SW52.1
- net Column10: now also SW10.1, SW38.1, SW61.1, SW24.1, U1.19 (20)
- net at SW52.2: now also D51.2 (A); no longer D48.2 (A)
- net Column12: now reaches SW54.1
- net Column12: now also SW12.1, SW40.1, SW63.1, SW26.1, U1.25 (1)
- net at D15.2 (A): now also SW19.2; no longer SW3.2
- net at D6.2 (A): now also SW5.2
- net at D17.2 (A): now also SW21.2; no longer SW5.2
- net at SW45.2: now also D44.2 (A)
- net Column5: now reaches SW33.1
- net Column5: now also SW47.1, SW5.1, SW19.1, U1.14 (16)
- net at D20.2 (A): now also SW24.2; no longer SW8.2
- net at SW50.2: now also D49.2 (A); no longer D50.2 (A)
- net at D21.2 (A): now also SW25.2; no longer SW9.2
- net Column1: now reaches SW56.1
- net Column1: now also SW1.1, SW15.1, SW43.1, SW29.1, U1.10 (7)
- net at SW16.2: now also D12.2 (A); no longer D56.2 (A)
- net at D35.2 (A): now also SW36.2; no longer SW38.2
- net at D41.2 (A): now also SW42.2; no longer SW32.2
- net at SW40.2: now also D39.2 (A); no longer D33.2 (A)
- net at SW57.2: now also D57.2 (A); no longer D43.2 (A)
- net at D4.2 (A): now also SW7.2
- net at SW49.2: now also D48.2 (A); no longer D51.2 (A)
- new net: D82.2 (A), SW28.2
- new net: D81.2 (A), SW27.2
- new net: D16.2 (A), SW20.2
- new net: D29.2 (A), SW30.2
- new net: D18.2 (A), SW22.2
- new net GND_lituam: BT1.2 (-)
- new net Sw1: J2.2 (Pin_2), On1.2 (B)
- new net VCC_lithuam: BT1.1 (+)
- no-connect marks 0 -> 5
Other:
- note added: "Keyboard Matrix"
- note added: "M3 Screws Holes"
- note added: "NiceNano"
- note added: "Oled"
- note added: "Power Managment"
- title: (none) -> Nonwire_Keyboard By youssef Ayman
- moved on the sheet: D23, D24, D25, D26, J1, SW10, SW11, SW12, SW13, SW14, SW2, SW3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
